File: PCB/BMU v1/BMU v1.kicad_sch (KiCad schematic)
At the start: 32 parts, among them J11 Screw_Terminal_01x01, J12 Screw_Terminal_01x01, J3 Conn_01x02_Pin, U8 VPS8505, U9 MCP16331T-E/CH

Commit message: update code
Connections:
- net GND: now also C12.2, C13.2, C19.2, C20.2, D1.2 (A), R25.2, U9.2 (GND)
- net GND_BATT: no longer C12.2, C13.2, C19.2, C20.2, D1.2 (A), R25.2, U9.2 (GND)
Changed lines of the file:
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@@
+	(wire
+		(pts
+			(xy 31.75 55.88) (xy 31.75 53.34)
+		)
+		(stroke
+			(width 0)
+			(type default)
+		)
+	)
 	(wire
 		(pts
@@
 		(pts
 			(xy 77.47 80.01) (xy 66.04 80.01)
-		)
-		(stroke
-			(width 0)
-			(type default)
-		)
-	)
-	(wire
-		(pts
-			(xy 31.75 63.5) (xy 31.75 53.34)
 		)
 		(stroke
@@
 			)
 			(justify right bottom)
-		)
-	)
-	(label "GND_BATT"
-		(at 31.75 63.5 90)
-		(fields_autoplaced yes)
-		(effects
-			(font
-				(size 1.27 1.27)
-			)
-			(justify left bottom)
 		)
 	)
@@
 					(unit 1)
 				)
+			)
+		)
+	)
+	(symbol
+		(lib_id "power:GND")
+		(at 31.75 55.88 0)
+		(unit 1)
+		(exclude_from_sim no)
+		(in_bom yes)
+		(on_board yes)
+		(dnp no)
+		(fields_autoplaced yes)
+		(property "Reference" "#PWR092"
+			(at 31.75 62.23 0)
+			(effects
+				(font
+					(size 1.27 1.27)
+				)
+				(hide yes)
+			)
+		)
+		(property "Value" "GND"
+			(at 31.75 60.325 0)
+			(effects
+				(font
+					(size 1.27 1.27)
+				)
+			)
+		)
+		(property "Footprint" ""
+			(at 31.75 55.88 0)
+			(effects
+				(font
+					(size 1.27 1.27)
+				)
+				(hide yes)
+			)
+		)
+		(property "Datasheet" ""
+			(at 31.75 55.88 0)
+			(effects
+				(font
+					(size 1.27 1.27)
+				)
+				(hide yes)
+			)
+		)
+		(property "Description" ""
+			(at 31.75 55.88 0)
+			(effects
+				(font
+					(size 1.27 1.27)
+				)
+				(hide yes)
+			)
+		)
+		(pin "1"
+		)
+		(instances
+			(project "BMU v1"
+				(path "/40c3f397-d07f-488b-b615-517efc4a5c8c"
+					(reference "#PWR092")
+					(unit 1)
+				)
