File: PCB BMU v2/BMU v2.kicad_pcb (KiCad board)
At the start: 4 copper layers, 193.5 x 105 mm, 143 parts, among them J1 RJ45_Shielded, J11 Screw_Terminal_01x01, J12 Screw_Terminal_01x01, J2 RJ45_Shielded, J3 Conn_01x02_Pin, Q5 IRFZ44NPBF, Q6 IRFZ44NPBF, Q7 IRFZ44NPBF, Q8 IRFZ44NPBF, U1 INA237, U10 MCP16331T-E/CH, U2 INA237, U3 INA237, U4 TCA9517ADGK, U5 ISO1540DR, U6 TCA9535PWR, U7 INA237, U8 VPS8505

Commit message: update code
Parts:
- removed D18, D19: 1A/100V, Diode_SMD:D_SMA
- removed the H13 at (165.0, 30.0)
- removed JP1: SolderJumper_2_Open, Jumper:SolderJumper-2_P1.3mm_Open_RoundedPad1.0x1.5mm
- removed R10, R11, R3, R4: 10R, Resistor_SMD:R_0603_1608Metric
- removed R13, R20, R40, R6: 470R, Resistor_THT:R_Axial_DIN0204_L3.6mm_D1.6mm_P5.08mm_Horizontal
- removed R14, R21, R41, R7: 10k, Resistor_THT:R_Axial_DIN0204_L3.6mm_D1.6mm_P5.08mm_Horizontal
- removed U10: MCP16331T-E/CH, Package_TO_SOT_SMD:SOT-23-6
- added C17: 20pF, Capacitor_SMD:C_0603_1608Metric, F.Cu at (6.66, 5.30)
- added D1: 1A/100V, Diode_SMD:D_SMA, F.Cu at (3.57, 1.77)
- added D13: 1N4148WT, Diode_SMD:D_SOD-523, F.Cu at (6.47, 7.79)
- added Q1: IRF4905STRLPBF, easyeda2kicad:D2PAK_L9.1-W10.0-P2.54-LS15.3-TL, F.Cu at (93.6, 223.0)
- added Q10: IRF4905STRLPBF, easyeda2kicad:D2PAK_L9.1-W10.0-P2.54-LS15.3-TL, F.Cu at (116.4, 234.6)
- added Q11: IRF4905STRLPBF, easyeda2kicad:D2PAK_L9.1-W10.0-P2.54-LS15.3-TL, F.Cu at (70.7, 234.6)
- added Q12: IRF4905STRLPBF, easyeda2kicad:D2PAK_L9.1-W10.0-P2.54-LS15.3-TL, F.Cu at (27.7, 224.0)
- added Q13: IRF4905STRLPBF, easyeda2kicad:D2PAK_L9.1-W10.0-P2.54-LS15.3-TL, F.Cu at (93.6, 246.1)
- added Q14: IRF4905STRLPBF, easyeda2kicad:D2PAK_L9.1-W10.0-P2.54-LS15.3-TL, F.Cu at (116.4, 246.1)
- added Q15: IRF4905STRLPBF, easyeda2kicad:D2PAK_L9.1-W10.0-P2.54-LS15.3-TL, F.Cu at (70.7, 246.1)
- added Q16: IRF4905STRLPBF, easyeda2kicad:D2PAK_L9.1-W10.0-P2.54-LS15.3-TL, F.Cu at (28.9, 210.3)
- added Q17: IRF4905STRLPBF, easyeda2kicad:D2PAK_L9.1-W10.0-P2.54-LS15.3-TL, F.Cu at (93.6, 257.7)
- added Q18: IRF4905STRLPBF, easyeda2kicad:D2PAK_L9.1-W10.0-P2.54-LS15.3-TL, F.Cu at (93.6, 269.3)
- added Q19: IRF4905STRLPBF, easyeda2kicad:D2PAK_L9.1-W10.0-P2.54-LS15.3-TL, F.Cu at (93.6, 280.9)
- added Q2: IRF4905STRLPBF, easyeda2kicad:D2PAK_L9.1-W10.0-P2.54-LS15.3-TL, F.Cu at (116.4, 223.0)
- added Q20: IRF4905STRLPBF, easyeda2kicad:D2PAK_L9.1-W10.0-P2.54-LS15.3-TL, F.Cu at (93.6, 292.4)
- added Q21: IRF4905STRLPBF, easyeda2kicad:D2PAK_L9.1-W10.0-P2.54-LS15.3-TL, F.Cu at (116.4, 257.7)
- added Q22: IRF4905STRLPBF, easyeda2kicad:D2PAK_L9.1-W10.0-P2.54-LS15.3-TL, F.Cu at (116.4, 269.3)
- added Q23: IRF4905STRLPBF, easyeda2kicad:D2PAK_L9.1-W10.0-P2.54-LS15.3-TL, F.Cu at (116.4, 280.9)
- added Q24: IRF4905STRLPBF, easyeda2kicad:D2PAK_L9.1-W10.0-P2.54-LS15.3-TL, F.Cu at (116.4, 292.4)
- added Q25: IRF4905STRLPBF, easyeda2kicad:D2PAK_L9.1-W10.0-P2.54-LS15.3-TL, F.Cu at (70.7, 257.7)
- added Q26: IRF4905STRLPBF, easyeda2kicad:D2PAK_L9.1-W10.0-P2.54-LS15.3-TL, F.Cu at (70.7, 269.3)
- added Q27: IRF4905STRLPBF, easyeda2kicad:D2PAK_L9.1-W10.0-P2.54-LS15.3-TL, F.Cu at (70.7, 280.9)
- added Q28: IRF4905STRLPBF, easyeda2kicad:D2PAK_L9.1-W10.0-P2.54-LS15.3-TL, F.Cu at (70.7, 292.4)
- added Q29: IRF4905STRLPBF, easyeda2kicad:D2PAK_L9.1-W10.0-P2.54-LS15.3-TL, F.Cu at (48.7, 188.0)
- added Q3: IRF4905STRLPBF, easyeda2kicad:D2PAK_L9.1-W10.0-P2.54-LS15.3-TL, F.Cu at (70.7, 223.0)
- added Q30: IRF4905STRLPBF, easyeda2kicad:D2PAK_L9.1-W10.0-P2.54-LS15.3-TL, F.Cu at (48.7, 199.6)
- added Q31: IRF4905STRLPBF, easyeda2kicad:D2PAK_L9.1-W10.0-P2.54-LS15.3-TL, F.Cu at (48.7, 211.1)
- added Q32: IRF4905STRLPBF, easyeda2kicad:D2PAK_L9.1-W10.0-P2.54-LS15.3-TL, F.Cu at (48.7, 222.7)
- added Q4: IRF4905STRLPBF, easyeda2kicad:D2PAK_L9.1-W10.0-P2.54-LS15.3-TL, F.Cu at (28.9, 185.0)
- added Q9: IRF4905STRLPBF, easyeda2kicad:D2PAK_L9.1-W10.0-P2.54-LS15.3-TL, F.Cu at (93.6, 234.6)
- added R42: 10K, Resistor_SMD:R_0603_1608Metric, F.Cu at (12.7, 0.76)
- added R43: 10K, Resistor_SMD:R_0603_1608Metric, F.Cu at (12.7, 3.27)
- added U9: MCP16331T-E/CH, Package_TO_SOT_SMD:SOT-23-6, F.Cu at (2.08, 6.45)
- C11, C3, C5, C7, C8, C9: footprint Capacitor_SMD:C_0805_2012Metric -> Capacitor_SMD:C_0402_1005Metric
- C12: value 1uF -> 10uF/50V; footprint Capacitor_SMD:C_0805_2012Metric -> Capacitor_SMD:C_1206_3216Metric
- C13: value 0,1uF -> 10uF/50V; footprint Capacitor_SMD:C_0805_2012Metric -> Capacitor_SMD:C_1206_3216Metric
- C14: value 10uF -> 0.1uF; footprint Capacitor_SMD:C_0805_2012Metric -> Capacitor_SMD:C_0603_1608Metric
- C15: value 10uF/50V -> 0,1uF; footprint Capacitor_SMD:C_1206_3216Metric -> Capacitor_SMD:C_0805_2012Metric
- C16: value 10uF/50V -> 1uF; footprint Capacitor_SMD:C_1206_3216Metric -> Capacitor_SMD:C_0805_2012Metric
- C18: value 0.1uF -> 10uF; footprint Capacitor_SMD:C_0603_1608Metric -> Capacitor_SMD:C_0805_2012Metric
- C19: value 20pF -> 10uF; footprint Capacitor_SMD:C_0603_1608Metric -> Capacitor_SMD:C_0805_2012Metric
- C21: value 10uF -> 0.1uF; footprint Capacitor_SMD:C_0805_2012Metric -> Capacitor_SMD:C_0402_1005Metric
- D9: value 1N4148WT -> 1A/100V; footprint Diode_SMD:D_SOD-523 -> Diode_SMD:D_SMA
- Q5, Q6, Q7, Q8: value IRFZ44NPBF -> IRF4905STRLPBF; footprint Package_TO_SOT_THT:TO-220-3_Horizontal_TabUp -> easyeda2kicad:D2PAK_L9.1-W10.0-P2.54-LS15.3-TL; moved to F.Cu
- R15: value 52.3k/1% -> 50R
- R17, R18, R37, R38: value 10R -> 10K
- R22: value 10k/1% -> 50R
- R24: value 50R -> 52.3k/1%
- R25: value 50R -> 10k/1%
- moved R38 188.7 mm to (40.2, 182.6), turned to 0 degrees
- moved R37 180.2 mm to (82.1, 218.5)
- moved G*** 162.5 mm to (45.5, 152.2)
- moved Q5 162.2 mm to (146.3, 250.4), turned to 0 degrees
- moved Q6 154.3 mm to (167.9, 250.4), turned to 0 degrees
- moved R17 148.8 mm to (105.0, 218.5)
- moved R18 145.0 mm to (127.8, 218.5), turned to 0 degrees
- moved Q8 129.5 mm to (146.3, 226.4), turned to 0 degrees
- moved Q7 121.6 mm to (167.9, 226.4), turned to 0 degrees
- moved D15 49.3 mm to (154.6, 97.5), turned to 180 degrees
- moved C11 44.9 mm to (159.0, 79.5)
- moved R39 44.4 mm to (154.3, 100.3)
- moved D16 44.3 mm to (159.6, 85.5), turned to 90 degrees
- moved D14 44.1 mm to (158.4, 97.5), turned to 0 degrees
- moved H14 43.6 mm to (132.0, 93.5)
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Connections:
- net /PCA_A0 renamed /I2C/PCA_A0
- net /PCA_A1 renamed /I2C/PCA_A1
- net /PCA_A2 renamed /I2C/PCA_A2
- net /SCL1 renamed /I2C/SCL1
- net /SDA1 renamed /I2C/SDA1
- C12 pad 1: +3.3V -> Net-(J3-Pin_2)
- C13 pad 1: +3.3V -> Net-(J3-Pin_2)
- C14 pad 1: +3.3V -> Net-(D13-K)
- C14 pad 2: GND -> Net-(D1-K)
- C15 pad 1: Net-(J3-Pin_2) -> +3.3V
- C15 pad 2: /GND_BATT -> GND
- C16 pad 1: Net-(J3-Pin_2) -> +3.3V
- C16 pad 2: /GND_BATT -> GND
- C18 pad 1: Net-(D9-K) -> +3.3V
- C18 pad 2: Net-(D5-K) -> GND
- C19 pad 2: Net-(U10-VFB) -> GND
- C20 pad 2: /GND_BATT -> GND
- C21 pad 1: /MANUAL_SW -> +3.3V
- C21 pad 2: /GND_BATT -> GND
- D12 pad 1: /batteries3/GND_BAT -> GND
- D16 pad 1: /batteries4/GND_BAT -> GND
- D20 pad 1: Net-(D20-K) -> GND
- D20 pad 2: GND -> Net-(D20-A)
- D21 pad 1: Net-(D21-K) -> GND
- D21 pad 2: GND -> Net-(D21-A)
- D22 pad 1: Net-(D22-K) -> GND
- D22 pad 2: GND -> Net-(D22-A)
- D23 pad 1: Net-(D23-K) -> GND
- D23 pad 2: GND -> Net-(D23-A)
- D24 pad 1: Net-(D24-K) -> GND
- D24 pad 2: GND -> Net-(D24-A)
- D25 pad 1: Net-(D25-K) -> GND
- D25 pad 2: GND -> Net-(D25-A)
- D26 pad 1: Net-(D26-K) -> GND
- D26 pad 2: GND -> Net-(D26-A)
- D27 pad 1: Net-(D27-K) -> GND
- D27 pad 2: GND -> Net-(D27-A)
- D4 pad 1: /GND_BATT -> GND
- D5 pad 1: Net-(D5-K) -> +3.3V
- D5 pad 2: /GND_BATT -> Net-(D5-A)
- D8 pad 1: /batteries2/GND_BAT -> GND
- D9 pad 1: Net-(D9-K) -> +3.3V
- D9 pad 2: /MANUAL_SW -> Net-(D9-A)
- H1 pad 1: /GND_BATT -> GND
- H11 pad 1: /batteries1/-BATT OUT -> GND
- H2 pad 1: /batteries2/GND_BAT -> GND
- H3 pad 1: /batteries3/GND_BAT -> GND
- H4 pad 1: /batteries4/GND_BAT -> GND
- J11 pad 2: +BATT -> (no net)
- J11 pad 3: +BATT -> (no net)
- J11 pad 4: +BATT -> (no net)
- J12 pad 1: /batteries1/-BATT OUT -> GND
- J12 pad 2: /batteries1/-BATT OUT -> (no net)
- J12 pad 3: /batteries1/-BATT OUT -> (no net)
- J12 pad 4: /batteries1/-BATT OUT -> (no net)
- L1 pad 1: Net-(D5-K) -> Net-(D1-K)
- Q5 pad 1: /batteries1/GATE -> Net-(Q1-G)
- Q5 pad 3: /GND_BATT -> Net-(Q1-S)
- Q6 pad 1: /batteries2/GATE -> Net-(Q10-G)
- Q6 pad 3: /batteries2/GND_BAT -> Net-(Q10-S)
- Q7 pad 1: /batteries3/GATE -> Net-(Q11-G)
- Q7 pad 3: /batteries3/GND_BAT -> Net-(Q11-S)
- Q8 pad 1: /batteries4/GATE -> Net-(Q12-G)
- Q8 pad 3: /batteries4/GND_BAT -> Net-(Q12-S)
- R1 pad 2: +BATT -> Net-(Q1-S)
- R1 pad 3: Net-(R1-Pad3) -> Net-(U1-Vin+)
- R1 pad 4: Net-(R1-Pad4) -> Net-(U1-Vin-)
- R15 pad 1: /MANUAL_SW -> Net-(R15-Pad1)
- R15 pad 2: Net-(U10-VFB) -> Net-(U8-VD2)
- R16 pad 1: Net-(J2-LEDG+) -> Net-(J2-LEDY+)
- R16 pad 2: VCC -> Net-(R16-Pad2)
- R17 pad 1: Net-(R17-Pad1) -> +3.3V
- R17 pad 2: Net-(U3-Vin+) -> /ALERT_1
- R18 pad 1: Net-(U3-Vin-) -> +3.3V
- R18 pad 2: Net-(R18-Pad2) -> /ALERT_2
- R22 pad 1: Net-(U10-VFB) -> Net-(R22-Pad1)
- R22 pad 2: /GND_BATT -> Net-(U8-VD1)
- R23 pad 1: Net-(J2-LEDY+) -> Net-(J2-LEDG+)
- R23 pad 2: Net-(R23-Pad2) -> VCC
- R24 pad 1: Net-(R24-Pad1) -> /MANUAL_SW
- R24 pad 2: Net-(U8-VD2) -> Net-(U9-VFB)
- R25 pad 1: Net-(R25-Pad1) -> Net-(U9-VFB)
- R25 pad 2: Net-(U8-VD1) -> GND
- R29 pad 1: Net-(D20-K) -> Net-(D20-A)
- R30 pad 1: Net-(D21-K) -> Net-(D21-A)
- R31 pad 1: Net-(D22-K) -> Net-(D22-A)
- R32 pad 1: Net-(D23-K) -> Net-(D23-A)
- R33 pad 1: Net-(D24-K) -> Net-(D24-A)
- R34 pad 1: Net-(D25-K) -> Net-(D25-A)
- R35 pad 1: Net-(D26-K) -> Net-(D26-A)
- R36 pad 1: Net-(D27-K) -> Net-(D27-A)
- R37 pad 1: Net-(R37-Pad1) -> +3.3V
- R37 pad 2: Net-(U7-Vin+) -> /ALERT_3
- R38 pad 1: Net-(U7-Vin-) -> +3.3V
- R38 pad 2: Net-(R38-Pad2) -> /ALERT_4
- R46 pad 2: +BATT -> Net-(Q11-S)
- R46 pad 3: Net-(R17-Pad1) -> Net-(U3-Vin+)
- R46 pad 4: Net-(R18-Pad2) -> Net-(U3-Vin-)
- R47 pad 2: +BATT -> Net-(Q12-S)
- R47 pad 3: Net-(R37-Pad1) -> Net-(U7-Vin+)
- R47 pad 4: Net-(R38-Pad2) -> Net-(U7-Vin-)
- R8 pad 2: +BATT -> Net-(Q10-S)
- R8 pad 3: Net-(R10-Pad1) -> Net-(U2-Vin+)
- R8 pad 4: Net-(R11-Pad2) -> Net-(U2-Vin-)
- TR1 pad 1: Net-(R24-Pad1) -> Net-(R15-Pad1)
- TR1 pad 3: Net-(R25-Pad1) -> Net-(R22-Pad1)
- TR1 pad 4: Net-(D19-A) -> Net-(D9-A)
- TR1 pad 6: Net-(D18-A) -> Net-(D5-A)
- U8 pad 5: Net-(JP1-B) -> VCC
Routing:
- net /MANUAL_SW: track 426.5 -> 41.7 mm, vias 8 -> 3
- net /SDA: track 372.4 -> 26.3 mm, vias 14 -> 1
- net +3.3V: track 398.1 -> 135.3 mm, vias 8 -> 1
- net /SCL: track 384.1 -> 134.4 mm, vias 14 -> 6
- net /GND_BATT: track 227.6 -> 0.00 mm, vias 1 -> 0
- net /BATT_SW4: track 213.3 -> 6.44 mm, vias 3 -> 1
- net /ALERT_4: track 202.7 -> 6.09 mm, vias 3 -> 1
- net GND: track 174.4 -> 0.00 mm, vias 19 -> 8
- net /BATT_SW3: track 179.3 -> 5.71 mm, vias 3 -> 1
- net /ALERT_3: track 155.1 -> 4.49 mm, vias 3 -> 1
- net /BATT_SW1: track 95.7 -> 36.1 mm, vias 3 -> 2
- net /BATT_SW2: track 138.2 -> 79.5 mm, vias 3 -> 2
- net /batteries1/-BATT OUT: track 52.7 -> 0.00 mm, vias 99 -> 0
- net Net-(J3-Pin_2): track 44.3 -> 0.00 mm
- net /ALERT_2: track 116.7 -> 77.4 mm, vias 3 -> 2
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- removed copper zone on B.Cu, net /GND_BATT
- removed copper zone on F.Cu, net /GND_BATT
- removed copper zone on In1.Cu, net /GND_BATT
- removed copper zone on In2.Cu, net /GND_BATT
- removed copper zone on B.Cu, net /batteries1/-BATT OUT
- removed copper zone on F.Cu, net /batteries1/-BATT OUT
- removed copper zone on In1.Cu, net /batteries1/-BATT OUT
- removed copper zone on In2.Cu, net /batteries1/-BATT OUT
- removed copper zone on B.Cu, net /batteries2/GND_BAT
- removed copper zone on F.Cu, net /batteries2/GND_BAT
- removed copper zone on In1.Cu, net /batteries2/GND_BAT
- removed copper zone on In2.Cu, net /batteries2/GND_BAT
- removed copper zone on B.Cu, net /batteries3/GND_BAT
- removed copper zone on F.Cu, net /batteries3/GND_BAT
- removed copper zone on In1.Cu, net /batteries3/GND_BAT
- removed copper zone on In2.Cu, net /batteries3/GND_BAT
- removed copper zone on B.Cu, net /batteries4/GND_BAT
- removed copper zone on F.Cu, net /batteries4/GND_BAT
- removed copper zone on In1.Cu, net /batteries4/GND_BAT
- removed copper zone on In2.Cu, net /batteries4/GND_BAT
Other:
- board size 193.5 x 105 mm -> 149.9 x 100 mm
- board text added: "${REFERENCE}"
- board text added: "Batterie Parallèlator v2 11/2024 Clément SAILLANT pour komplex kapharnaüm"
- board text removed: "Batterie Parallèlator v 0.1a 09/2024 Clément SAILLANT pour komplex kapharnaüm"

Commit message: PCB update
Parts:
- removed Q1, Q10, Q11, Q12, Q13, Q14, Q15, Q16, Q17, Q18, Q19, Q2, Q20, Q21, Q22, Q23, Q24, Q25, Q26, Q27, Q28, Q29, Q3, Q30, Q31, Q32, Q4, Q5, Q6, Q7, Q8, Q9: IRF4905STRLPBF, easyeda2kicad:D2PAK_L9.1-W10.0-P2.54-LS15.3-TL
- added H15: FH-00020, easyeda2kicad:HDR-TH_10P-P2.54-V-F-R2-C5-S2.54, B.Cu at (51.7, 82.5)
- added H16: FH-00020, easyeda2kicad:HDR-TH_10P-P2.54-V-F-R2-C5-S2.54, F.Cu at (50.4, 4.04)
- added H17: FH-00020, easyeda2kicad:HDR-TH_10P-P2.54-V-F-R2-C5-S2.54, F.Cu at (137.9, 144.8)
- added H18: FH-00020, easyeda2kicad:HDR-TH_10P-P2.54-V-F-R2-C5-S2.54, F.Cu at (19.6, 4.04)
- added H19: FH-00020, easyeda2kicad:HDR-TH_10P-P2.54-V-F-R2-C5-S2.54, F.Cu at (55.1, 65.3)
- added H20: FH-00020, easyeda2kicad:HDR-TH_10P-P2.54-V-F-R2-C5-S2.54, F.Cu at (137.9, 177.7)
- added H21: FH-00020, easyeda2kicad:HDR-TH_10P-P2.54-V-F-R2-C5-S2.54, F.Cu at (137.9, 153.9)
- added H22: FH-00020, easyeda2kicad:HDR-TH_10P-P2.54-V-F-R2-C5-S2.54, F.Cu at (64.9, 162.7)
- added H23: 12251103CNG0S115001, easyeda2kicad:HDR-TH_3P-P2.54-V-M-1, F.Cu at (76.0, 79.5)
- added H24: 12251103CNG0S115001, easyeda2kicad:HDR-TH_3P-P2.54-V-M-1, F.Cu at (49.3, -26.3)
- added H25: 12251103CNG0S115001, easyeda2kicad:HDR-TH_3P-P2.54-V-M-1, F.Cu at (38.5, -26.3)
- added H26: 12251103CNG0S115001, easyeda2kicad:HDR-TH_3P-P2.54-V-M-1, F.Cu at (38.5, -32.0)
- JP2, JP3, JP4, JP5: moved to B.Cu
- moved R17 198.7 mm to (109.3, 19.8)
- moved R18 198.7 mm to (132.2, 19.8)
- moved R37 198.7 mm to (86.5, 19.8)
- moved U9 169.7 mm to (168.2, 40.7)
- moved C17 169.7 mm to (172.8, 39.5)
- moved D1 169.7 mm to (169.7, 36.0)
- moved D13 169.7 mm to (172.6, 42.0)
- moved R42 169.7 mm to (178.8, 35.0)
- moved R43 169.7 mm to (178.8, 37.5)
- moved JP17 159.3 mm to (13.9, 19.6), turned to 0 degrees
- moved H8 158.7 mm to (5.28, 16.8)
- moved D14 158.2 mm to (18.5, 23.6)
- moved JP19 157.4 mm to (13.9, 26.7), turned to 0 degrees
- moved JP18 156.6 mm to (13.9, 23.1), turned to 0 degrees
- moved D15 153.7 mm to (18.5, 26.0), turned to 0 degrees
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Connections:
- net Net-(D10-K) renamed /batteries3/CMD_Switch_bat
- net Net-(D14-K) renamed /batteries4/CMD_Switch_bat
- net Net-(D2-K) renamed /batteries1/CMD_Switch_bat
- net Net-(D6-K) renamed /batteries2/CMD_Switch_bat
- R1 pad 2: Net-(Q1-S) -> /batteries1/+BATT_SHUNT_OUT
- R46 pad 2: Net-(Q11-S) -> /batteries3/+BATT_SHUNT_OUT
- R47 pad 2: Net-(Q12-S) -> /batteries4/+BATT_SHUNT_OUT
- R8 pad 2: Net-(Q10-S) -> /batteries2/+BATT_SHUNT_OUT
Routing:
- net +3.3V: track 135.3 -> 406.8 mm, vias 1 -> 4
- net /SCL: track 134.4 -> 375.4 mm, vias 6 -> 20
- net /SDA: track 26.3 -> 254.2 mm, vias 1 -> 10
- net /BATT_SW3: track 5.71 -> 77.6 mm, vias 1 -> 4
- net /BATT_SW2: track 79.5 -> 150.0 mm, vias 2 -> 5
- net GND: track 0.00 -> 59.2 mm, vias 8 -> 21
- net Net-(D22-A): track 0.00 -> 57.7 mm, vias 0 -> 2
- net /ALERT_1: track 41.6 -> 86.5 mm, vias 2 -> 3
- net /BATT_SW1: track 36.1 -> 79.6 mm, vias 2 -> 4
- net /ALERT_2: track 77.4 -> 117.6 mm, vias 2 -> 4
- net /BATT_SW4: track 6.44 -> 45.2 mm, vias 1 -> 3
- net /ALERT_3: track 4.49 -> 42.7 mm, vias 1 -> 3
- net +BATT: track 0.00 -> 34.1 mm
- net /batteries2/+BAT_IN: track 0.00 -> 27.7 mm
- net /batteries3/+BAT_IN: track 0.00 -> 18.3 mm
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- added copper zone on B.Cu, net /batteries1/+BATT_SHUNT_OUT
- added copper zone on F.Cu, net /batteries1/+BATT_SHUNT_OUT
- added copper zone on In1.Cu, net /batteries1/+BATT_SHUNT_OUT
- added copper zone on In2.Cu, net /batteries1/+BATT_SHUNT_OUT
- added copper zone on B.Cu, net /batteries2/+BATT_SHUNT_OUT
- added copper zone on F.Cu, net /batteries2/+BATT_SHUNT_OUT
- added copper zone on In1.Cu, net /batteries2/+BATT_SHUNT_OUT
- added copper zone on In2.Cu, net /batteries2/+BATT_SHUNT_OUT
- added copper zone on B.Cu, net /batteries3/+BATT_SHUNT_OUT
- added copper zone on F.Cu, net /batteries3/+BATT_SHUNT_OUT
- added copper zone on In1.Cu, net /batteries3/+BATT_SHUNT_OUT
- added copper zone on In2.Cu, net /batteries3/+BATT_SHUNT_OUT
- added copper zone on B.Cu, net /batteries4/+BATT_SHUNT_OUT
- added copper zone on F.Cu, net /batteries4/+BATT_SHUNT_OUT
- added copper zone on In1.Cu, net /batteries4/+BATT_SHUNT_OUT
- added copper zone on In2.Cu, net /batteries4/+BATT_SHUNT_OUT
Other:
- board size 149.9 x 100 mm -> 194.9 x 100 mm
- board text removed: "${REFERENCE}"
- board text removed: "ON"

Commit message: add Ampère/Houre calculation
Parts:
- removed C1: 10uF,16V, Capacitor_SMD:CP_Elec_8x10
- removed C15: 0,1uF, Capacitor_SMD:C_0805_2012Metric
- removed C16: 1uF, Capacitor_SMD:C_0805_2012Metric
- removed C18: 10uF, Capacitor_SMD:C_0805_2012Metric
- removed C21, C8: 0.1uF, Capacitor_SMD:C_0402_1005Metric
- removed D5, D9: 1A/100V, Diode_SMD:D_SMA
- removed the H1 at (57.9, 114.0)
- removed H10, H13, H14, H9: MountingHole, MountingHole:MountingHole_3.2mm_M3_DIN965
- removed H11, H12: MountingHole_Pad, MountingHole:MountingHole_3.2mm_M3_Pad_Via
- removed the H2 at (36.0, 5.28)
- removed J2: RJ45_Shielded, easyeda2kicad:RJ45-TH_RC01061
- removed R15, R22: 50R, Resistor_SMD:R_0603_1608Metric
- removed R16, R2, R23, R9: 470R, Resistor_SMD:R_0603_1608Metric
- removed R26, R27: 1K, Resistor_SMD:R_0603_1608Metric
- removed R42, R43: 10K, Resistor_SMD:R_0603_1608Metric
- removed TR1: VPT85BB-01A, Transformer_SMD:VP85BB-01A
- removed U4: TCA9517ADGK, easyeda2kicad:VSSOP-8_L3.0-W3.0-P0.65-LS5.0-BL
- removed U5: ISO1540DR, Package_SO:SOIC-8_3.9x4.9mm_P1.27mm
- removed U8: VPS8505, easyeda2kicad:SOT-23-6_L2.9-W1.6-P0.95-LS2.8-BR
- added H1: MountingHole_Pad, MountingHole:MountingHole_5mm_Pad, F.Cu at (57.2, 112.0)
- added H1: MountingHole_Pad, MountingHole:MountingHole_5mm_Pad, F.Cu at (22.3, 49.2)
- added H1: MountingHole_Pad, MountingHole:MountingHole_5mm_Pad, F.Cu at (23.0, 26.8)
- added H2: MountingHole_Pad, MountingHole:MountingHole_5mm_Pad, F.Cu at (61.3, 26.8)
- added H2: MountingHole_Pad, MountingHole:MountingHole_5mm_Pad, F.Cu at (96.3, 112.0)
- added HM1: MountingHole, MountingHole:MountingHole_2.7mm_M2.5, B.Cu at (61.5, 79.5)
- added HM2: MountingHole, MountingHole:MountingHole_2.7mm_M2.5, B.Cu at (100.5, 79.6)
- added HM3: MountingHole, MountingHole:MountingHole_2.7mm_M2.5, B.Cu at (139.6, 79.5)
- added HM4: MountingHole, MountingHole:MountingHole_2.7mm_M2.5, B.Cu at (178.5, 79.5)
- H16, H17, H18, H19, H20, H21, H22, H23, H24, H25, H26, JP10, JP11, JP12, JP13, JP14, JP15, JP16, JP17, JP18, JP19, JP20, JP6, JP7, JP8, JP9: moved to B.Cu
- J1: value RJ45_Shielded -> Conn_01x04; footprint easyeda2kicad:RJ45-TH_RC01061 -> Connector_PinSocket_2.54mm:PinSocket_1x04_P2.54mm_Vertical
- J11, J12: value Screw_Terminal_01x01 -> T68160200-1300
- L1: value 22uH,1.5A -> SLW5040S220MST; footprint Inductor_SMD:L_Taiyo-Yuden_NR-50xx -> easyeda2kicad:IND-SMD_L5.0-W5.0
- moved H8 196.2 mm to (179.0, 108.0)
- moved H26 183.1 mm to (177.4, 87.3), turned to 180 degrees
- moved R38 178.9 mm to (179.8, 50.8)
- moved JP17 176.5 mm to (183.7, 67.7)
- moved JP19 175.4 mm to (183.7, 70.5)
- moved U7 174.9 mm to (184.0, 82.0), turned to -90 degrees
- moved JP18 174.9 mm to (183.7, 65.0)
- moved R47 173.9 mm to (173.2, 94.0), turned to 180 degrees
- moved JP20 172.8 mm to (183.7, 62.3)
- moved C10 172.6 mm to (183.0, 87.5), turned to 180 degrees
- moved D14 171.1 mm to (182.0, 74.0), turned to 90 degrees
- moved H18 168.4 mm to (168.7, 82.6), turned to 90 degrees
- moved D16 165.9 mm to (178.0, 84.0), turned to 180 degrees
- moved C11 164.9 mm to (181.0, 84.5), turned to -90 degrees
- moved D15 164.3 mm to (175.0, 76.0), turned to 90 degrees
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Connections:
- H5 pad 1: /batteries1/+BAT_IN -> /Batt_SW
- J1 pad 1: GND1 -> +3.3V
- J1 pad 2: GND1 -> /SCL
- J1 pad 3: Net-(U4-SDAA) -> /SDA
- J1 pad 4: Net-(U4-SCLA) -> GND
- J11 pad 2: (no net) -> +BATT
- J11 pad 3: (no net) -> +BATT
- J11 pad 4: (no net) -> +BATT
- J12 pad 2: (no net) -> GND
- J12 pad 3: (no net) -> GND
- J12 pad 4: (no net) -> GND
- J3 pad 1: +BATT -> /Batt_SW
- R1 pad 1: /batteries1/+BAT_IN -> /Batt_SW
- U1 pad 8: /batteries1/+BAT_IN -> /Batt_SW
Routing:
- net /MANUAL_SW: track 45.9 -> 279.8 mm, vias 7 -> 6
- net /Batt_SW: track 0.00 -> 213.9 mm
- net VCC: track 128.0 -> 0.00 mm
- net /BATT_SW2: track 150.0 -> 39.1 mm, vias 5 -> 2
- net /ALERT_4: track 6.09 -> 103.4 mm, vias 1 -> 3
- net /ALERT_2: track 117.6 -> 59.4 mm, vias 4 -> 3
- net Net-(D22-A): track 57.7 -> 2.40 mm, vias 2 -> 0
- net /SCL: track 375.4 -> 320.2 mm, vias 20 -> 8
- net /BATT_SW4: track 45.2 -> 96.5 mm, vias 3 -> 2
- net /ALERT_3: track 42.7 -> 93.2 mm, vias 3 -> 4
- net /SDA: track 254.2 -> 300.4 mm, vias 10 -> 9
- net +BATT: track 34.1 -> 0.00 mm, vias 0 -> 674
- net /I2C/PCA_A0: track 0.00 -> 32.9 mm, vias 0 -> 1
- net Net-(U6-P14): track 44.3 -> 12.8 mm
- net Net-(U6-P16): track 58.3 -> 26.9 mm
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- added copper zone on B.Cu, net /Batt_SW
- added copper zone on F.Cu, net /Batt_SW
- added copper zone on In1.Cu, net /Batt_SW
- added copper zone on In2.Cu, net /Batt_SW
- removed copper zone on B.Cu, net /batteries1/+BAT_IN
- removed copper zone on F.Cu, net /batteries1/+BAT_IN
- removed copper zone on In1.Cu, net /batteries1/+BAT_IN
- removed copper zone on In2.Cu, net /batteries1/+BAT_IN
- removed copper zone on B.Cu, net GND1
- removed copper zone on F.Cu, net GND1
- removed copper zone on In1.Cu, net GND1
- removed copper zone on In2.Cu, net GND1
Other:
- board size 194.9 x 100 mm -> 170 x 100 mm
- board text added: "AO"
- board text added: "BATT 1"
- board text added: "BATT 1 +"
- board text added: "BATT 1 -"
- board text added: "BATT 2"
- board text added: "BATT 2 +"
- board text added: "BATT 2 -"
- board text added: "BATT 3"
- board text added: "BATT 3 +"
- board text added: "BATT 3 -"
- board text added: "BATT 4"
- board text added: "BATT 4 +"
- board text added: "BATT 4 -"
- board text added: "Batterie 1"
- board text added: "Batterie 2"
- board text added: "Batterie 3"
- board text added: "Batterie 4"
- board text added: "GND"
- board text added: "GND SDA SCL VCC"
- board text added: "I2C Board"
- board text added: "SCL"
- board text added: "SDA"
- board text added: "VCC"
- board text added: "VCC / GND"
- board text removed: "Batt 1"
- board text removed: "Batt 2"
- board text removed: "Batt 3"
- board text removed: "Batt 4"
- board text removed: "Batterie Parallèlator v2 11/2024 Clément SAILLANT pour komplex kapharnaüm"
- board text removed: "ENABLE"
- board text removed: "INPUT"
- board text removed: "OUTPUT"
- board text removed: "Switch Manual ON"
- board text removed: "VCC/GND"
