File: PCB BMU v2/BMU-v2/BMU v2.kicad_pcb (KiCad board)
At the start: 4 copper layers, 170 x 100 mm, 142 parts, among them J1 Conn_01x04, J11 T68160200-1300, J12 T68160200-1300, J2 RJ45_Shielded, J3 Conn_01x02_Pin, J4 RJ45_Shielded, J5 Conn_01x02_Pin, U1 INA237, U2 INA237, U3 INA237, U4 VPS8505, U6 TCA9535PWR, U7 INA237, U8 ISO1540DR, U9 MCP16331T-E/CH

Commit message: update PCB
Parts:
- removed J2, J4: RJ45_Shielded, easyeda2kicad:RJ45-TH_RC02535
- added R1: 470R, Resistor_SMD:R_0603_1608Metric, F.Cu at (66.5, 81.2)
- added R20: 470R, Resistor_SMD:R_0603_1608Metric, F.Cu at (144.4, 81.2)
- added R21: 470R, Resistor_SMD:R_0603_1608Metric, F.Cu at (180.5, 75.1)
- added R8: 470R, Resistor_SMD:R_0603_1608Metric, F.Cu at (105.2, 81.4)
- added RJ1: RC02113, easyeda2kicad:RJ45-TH_RC02113, F.Cu at (62.5, 33.6)
- added RJ2: RC02113, easyeda2kicad:RJ45-TH_RC02113, F.Cu at (43.4, 33.6)
- R12, R19, R39, R5: value 470R -> 22R
- moved HM4 5.00 mm to (25.0, 116.0)
- moved HM4 5.00 mm to (25.0, 26.0)
- moved D15 0.60 mm to (176.2, 75.1)
- moved D16 0.60 mm to (178.0, 84.6)
- moved D14 0.41 mm to (182.4, 73.5)
Connections:
- D10 pad 1: /batteries3/CMD_Switch_bat -> Net-(D10-K)
- D10 pad 2: /BATT_SW3 -> /MANUAL_SW
- D11 pad 2: /MANUAL_SW -> /BATT_SW3
- D14 pad 1: /batteries4/CMD_Switch_bat -> Net-(D14-K)
- D14 pad 2: /BATT_SW4 -> /MANUAL_SW
- D15 pad 2: /MANUAL_SW -> /BATT_SW4
- D2 pad 1: /batteries1/CMD_Switch_bat -> Net-(D2-K)
- D2 pad 2: /BATT_SW1 -> /MANUAL_SW
- D3 pad 2: /MANUAL_SW -> /BATT_SW1
- D6 pad 1: /batteries2/CMD_Switch_bat -> Net-(D6-K)
- D6 pad 2: /BATT_SW2 -> /MANUAL_SW
- D7 pad 2: /MANUAL_SW -> /BATT_SW2
Routing:
- net /BATT_SW4: track 94.7 -> 101.4 mm
- net /MANUAL_SW: track 274.9 -> 269.6 mm
- net /BATT_SW1: track 75.8 -> 71.8 mm
- net Net-(D6-K): track 0.00 -> 3.13 mm
- net Net-(D10-K): track 0.00 -> 3.08 mm
- net Net-(D2-K): track 0.00 -> 2.83 mm
- net /BATT_SW3: track 76.9 -> 74.2 mm
- net /BATT_SW2: track 38.9 -> 36.4 mm
- net Net-(D14-K): track 0.00 -> 2.19 mm
- net /batteries1/CMD_Switch_bat: track 15.3 -> 14.0 mm
- net /batteries3/CMD_Switch_bat: track 15.3 -> 14.0 mm
- net /batteries2/CMD_Switch_bat: track 15.0 -> 14.0 mm
- net /batteries4/CMD_Switch_bat: track 21.0 -> 20.0 mm
Other:
- outline, holes or cut-outs redrawn
