File: PCB BMU v2/BMU-v2/batteries.kicad_sch (KiCad schematic)
At the start: 18 parts, among them U7 INA237

Commit message: update PCB
Parts:
- added R21: 470R, Resistor_SMD:R_0603_1608Metric, symbol Device:R_Small
- R39: value 470R -> 22R
- renumbered R10 to R14
Connections:
- net BATT_SW: now also D15.2 (A); no longer D14.2 (A)
- net CMD_Switch_bat: now also R21.1; no longer D14.1 (K)
- net MANUAL_SW: now also D14.2 (A); no longer D15.2 (A)
- new net: D14.1 (K), R21.2
Changed lines of the file:
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@@
 	(wire
 		(pts
-			(xy 151.13 36.83) (xy 151.13 49.53)
+			(xy 151.13 36.83) (xy 151.13 39.37)
 		)
 		(stroke
@@
 	(wire
 		(pts
+			(xy 151.13 44.45) (xy 151.13 49.53)
+		)
+		(stroke
+			(width 0)
+			(type default)
+		)
+	)
+	(wire
+		(pts
 			(xy 151.13 58.42) (xy 151.13 55.88)
 		)
@@
 	(hierarchical_label "MANUAL_SW"
 		(shape input)
-		(at 133.35 49.53 180)
+		(at 133.35 36.83 180)
 		(effects
 			(font
@@
 		)
 	)
-	(hierarchical_label "SDA"
-		(shape bidirectional)
-		(at 234.95 133.35 0)
+	(hierarchical_label "BATT_SW"
+		(shape input)
+		(at 133.35 49.53 180)
 		(effects
 			(font
 				(size 1.27 1.27)
 			)
-			(justify left)
+			(justify right)
 		)
 	)
-	(hierarchical_label "BATT_SW"
-		(shape input)
-		(at 133.35 36.83 180)
+	(hierarchical_label "SDA"
+		(shape bidirectional)
+		(at 234.95 133.35 0)
 		(effects
 			(font
 				(size 1.27 1.27)
 			)
-			(justify right)
+			(justify left)
 		)
 	)
@@
 		(dnp no)
 		(fields_autoplaced yes)
-		(property "Reference" "R10"
+		(property "Reference" "R14"
 			(at 180.34 137.1599 90)
 			(effects
@@
 			)
 		)
-		(property "Value" "470R"
+		(property "Value" "22R"
 			(at 152.781 53.34 90)
 			(effects
@@
 					(unit 1)
 				)
+			)
+		)
+	)
+	(symbol
+		(lib_id "Device:R_Small")
+		(at 151.13 41.91 180)
+		(unit 1)
+		(exclude_from_sim no)
+		(in_bom yes)
+		(on_board yes)
+		(dnp no)
+		(property "Reference" "R21"
+			(at 149.479 41.91 90)
+			(effects
+				(font
+					(size 1.27 1.27)
+				)
+			)
+		)
+		(property "Value" "470R"
+			(at 152.781 41.91 90)
+			(effects
+				(font
+					(size 1.27 1.27)
+				)
+			)
+		)
+		(property "Footprint" "Resistor_SMD:R_0603_1608Metric"
+			(at 151.13 41.91 0)
+			(effects
+				(font
+					(size 1.27 1.27)
+				)
+				(hide yes)
+			)
+		)
+		(property "Datasheet" "~"
+			(at 151.13 41.91 0)
+			(effects
+				(font
+					(size 1.27 1.27)
+				)
+				(hide yes)
+			)
+		)
+		(property "Description" ""
+			(at 151.13 41.91 0)
+			(effects
+				(font
+					(size 1.27 1.27)
+				)
+				(hide yes)
+			)
+		)
+		(pin "1"
+		)
+		(pin "2"
+		)
+		(instances
+			(project "BMU v2"
+				(path "/40c3f397-d07f-488b-b615-517efc4a5c8c/404fd779-052a-4b44-92bc-a9ff818e1713"
+					(reference "R21")
+					(unit 1)
+				)
+				(path "/40c3f397-d07f-488b-b615-517efc4a5c8c/8e75d9c9-36b3-4715-8008-0cb2c10c4fbe"
+					(reference "R20")
+					(unit 1)
+				)
+				(path "/40c3f397-d07f-488b-b615-517efc4a5c8c/9b15f43a-be76-42f8-a3fd-d61e4c342bdb"
+					(reference "R1")
+					(unit 1)
+				)
+				(path "/40c3f397-d07f-488b-b615-517efc4a5c8c/ede9b4b7-549c-4a0a-90de-aef8f304e75f"
+					(reference "R8")
+					(unit 1)
+				)
