File: PCB BMU v2/BMU_switch_mosfet/BMU_switch_mosfet.kicad_pcb (KiCad board)
At the start: 2 copper layers, 38 x 85.5 mm, 22 parts, among them Q1 BC847CLT1G, Q10 IRF4905STRLPBF, Q11 BC847CLT1G, Q2 IRF4905STRLPBF, Q3 IRF4905STRLPBF, Q4 IRF4905STRLPBF, Q5 IRF4905STRLPBF, Q7 IRF4905STRLPBF, Q8 IRF4905STRLPBF, Q9 IRF4905STRLPBF, U1 HX PZ2.54-1X2P ZZ, U2 ZX-IDC2.54-2-5PZZ, U3 ZX-IDC2.54-2-5PZZ

Commit message: update PCB
Parts:
- moved Q11 1.47 mm to (154.3, 148.2), turned to 90 degrees
Routing:
- net Net-(Q10-G): track 173.4 -> 167.2 mm, vias 6 -> 4
- net Net-(Q11-B): track 6.71 -> 4.71 mm
- net /CMD_Switch_bat: track 40.2 -> 41.6 mm
